Commit message: added gripper cam & colour to ur5

File: data/ur5/ur5_with_panda_gripper_long_finger.urdf (robot description, URDF)
Before this commit: robot ur5_robot, 16 links, 15 joints
Links:
- added link gripper_cam, mass 0.2; visual box size=.08 .025 0.01
- link panda_leftfinger: geometry collision mesh filename=package://meshes/collision/longer_finger_v2.obj scale=1.0 1.0 0.6; visual mesh filename=package://meshes/visual/longer_finger_v2.obj scale=1.0 1.0 0.6
- link panda_rightfinger: geometry collision mesh filename=package://meshes/collision/longer_finger_v2.obj scale=1.0 1.0 0.6; visual mesh filename=package://meshes/visual/longer_finger_v2.obj scale=1.0 1.0 0.6
Joints:
- added joint camera_joint: type fixed, parent panda_hand, child gripper_cam, origin xyz=-0.1 0 0 rpy=1.3  0 -1.57
- joint tcp_joint: origin xyz=0 0 0.1 rpy=0 0 3.14 -> xyz=0 0 0.1 rpy=0 0 0
